Commit message: debug: urdf and meshes

File: assets/abb_irb1200_509_gripper/irb1200.urdf (robot description, URDF)
Before this commit: robot abb_irb1200_5_90, 19 links, 18 joints
Links:
- link left_inner_finger: geometry collision mesh filename=assets\abb_irb1200_509_gripper\meshes_gripper\inner_finger_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; visual mesh filename=assets\abb_irb1200_509_gripper\meshes_gripper\inner_finger_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
- link left_inner_knuckle: geometry collision mesh filename=assets\abb_irb1200_509_gripper\meshes_gripper\inner_knuckle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; visual mesh filename=assets\abb_irb1200_509_gripper\meshes_gripper\inner_knuckle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
- link left_outer_finger: geometry collision mesh filename=assets\abb_irb1200_509_gripper\meshes_gripper\outer_finger_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; visual mesh filename=assets\abb_irb1200_509_gripper\meshes_gripper\outer_finger_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
- link left_outer_knuckle: geometry collision mesh filename=assets\abb_irb1200_509_gripper\meshes_gripper\outer_knuckle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; visual mesh filename=assets\abb_irb1200_509_gripper\meshes_gripper\outer_knuckle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
- link right_inner_finger: geometry collision mesh filename=assets\abb_irb1200_509_gripper\meshes_gripper\inner_finger_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; visual mesh filename=assets\abb_irb1200_509_gripper\meshes_gripper\inner_finger_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
- link right_inner_knuckle: geometry collision mesh filename=assets\abb_irb1200_509_gripper\meshes_gripper\inner_knuckle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; visual mesh filename=assets\abb_irb1200_509_gripper\meshes_gripper\inner_knuckle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
- link right_outer_finger: geometry collision mesh filename=assets\abb_irb1200_509_gripper\meshes_gripper\outer_finger_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; visual mesh filename=assets\abb_irb1200_509_gripper\meshes_gripper\outer_finger_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
- link right_outer_knuckle: geometry collision mesh filename=assets\abb_irb1200_509_gripper\meshes_gripper\outer_knuckle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; visual mesh filename=assets\abb_irb1200_509_gripper\meshes_gripper\outer_knuckle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
- link robotiq_85_base_link: geometry collision mesh filename=assets\abb_irb1200_509_gripper\meshes_gripper\robotiq_85_ba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; visual mesh filename=assets\abb_irb1200_509_gripper\meshes_gripper\robotiq_85_ba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

File: assets/abb_irb1200_509_gripper/irb1200_full.urdf (robot description, URDF)
Before this commit: robot abb_irb1200_5_90, 19 links, 18 joints
Links:
- link left_inner_finger: geometry collision mesh filename=assets\abb_irb1200_509_gripper\meshes_gripper\inner_finger_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; visual mesh filename=assets\abb_irb1200_509_gripper\meshes_gripper\inner_finger_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
- link left_inner_knuckle: geometry collision mesh filename=assets\abb_irb1200_509_gripper\meshes_gripper\inner_knuckle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; visual mesh filename=assets\abb_irb1200_509_gripper\meshes_gripper\inner_knuckle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
- link left_outer_finger: geometry collision mesh filename=assets\abb_irb1200_509_gripper\meshes_gripper\outer_finger_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; visual mesh filename=assets\abb_irb1200_509_gripper\meshes_gripper\outer_finger_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
- link left_outer_knuckle: geometry collision mesh filename=assets\abb_irb1200_509_gripper\meshes_gripper\outer_knuckle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; visual mesh filename=assets\abb_irb1200_509_gripper\meshes_gripper\outer_knuckle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
- link right_inner_finger: geometry collision mesh filename=assets\abb_irb1200_509_gripper\meshes_gripper\inner_finger_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; visual mesh filename=assets\abb_irb1200_509_gripper\meshes_gripper\inner_finger_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
- link right_inner_knuckle: geometry collision mesh filename=assets\abb_irb1200_509_gripper\meshes_gripper\inner_knuckle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; visual mesh filename=assets\abb_irb1200_509_gripper\meshes_gripper\inner_knuckle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
- link right_outer_finger: geometry collision mesh filename=assets\abb_irb1200_509_gripper\meshes_gripper\outer_finger_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; visual mesh filename=assets\abb_irb1200_509_gripper\meshes_gripper\outer_finger_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
- link right_outer_knuckle: geometry collision mesh filename=assets\abb_irb1200_509_gripper\meshes_gripper\outer_knuckle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; visual mesh filename=assets\abb_irb1200_509_gripper\meshes_gripper\outer_knuckle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
- link robotiq_85_base_link: geometry collision mesh filename=assets\abb_irb1200_509_gripper\meshes_gripper\robotiq_85_ba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; visual mesh filename=assets\abb_irb1200_509_gripper\meshes_gripper\robotiq_85_ba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
