Commit message: refactor: add dynamics to robot urdf and set limits for gripper

File: assets/abb_irb1200_509_gripper/irb1200_full.urdf (robot description, URDF)
Before this commit: robot abb_irb1200_5_90, 19 links, 18 joints
Joints:
- joint joint_1: limit lower=-2.967 upper=2.967 effort=0 velocity=5.027 -> lower=-2.967 upper=2.967 effort=1000 velocity=5.027
- joint joint_2: limit lower=-1.745 upper=2.269 effort=0 velocity=4.189 -> lower=-1.745 upper=2.269 effort=1000 velocity=4.189
- joint joint_3: limit lower=-3.491 upper=1.222 effort=0 velocity=5.236 -> lower=-3.491 upper=1.222 effort=1000 velocity=5.236
- joint joint_4: limit lower=-4.712 upper=4.712 effort=0 velocity=6.981 -> lower=-4.712 upper=4.712 effort=1000 velocity=6.981
- joint joint_5: limit lower=-2.269 upper=2.269 effort=0 velocity=7.069 -> lower=-2.269 upper=2.269 effort=1000 velocity=7.069
- joint joint_6: limit lower=-6.283 upper=6.283 effort=0 velocity=10.472 -> lower=-6.283 upper=6.283 effort=1000 velocity=10.472

Commit message: refactor: add inertia for base, tool0, robotiq_tcp and add colision for IK solver

File: assets/abb_irb1200_509_gripper/irb1200_full.urdf (robot description, URDF)
Before this commit: robot abb_irb1200_5_90, 19 links, 18 joints
Links:
- link base: mass None -> 0.001
- link robotiq_tcp: mass None -> 0.001
- link tool0: mass None -> 0.001
